Commit message: Initial Update to Indigo

File: turtlebot_le2i/urdf/rplidar.urdf.xacro (robot description, xacro)
@@ -5,5 +5,5 @@
 	<xacro:macro name="sensor_rplidar" params="parent">
   	<joint name="laser" type="fixed">
-		<origin xyz="0.180 0.00 0.040" rpy="0 3.14159265 0" />
+		<origin xyz="0.180 0.00 0.040" rpy="0 0 0" />
 		<parent link="${parent}" />
 		<child link="base_laser_link" />
@@ -11,15 +11,25 @@
 	<link name="base_laser_link">
 		<visual>
+			<origin xyz="-0.0425 0.035 -0.040" rpy="1.570796327 0 0"/>
 			<geometry>
-				<box size="0.00 0.05 0.06" />
+				<mesh filename="package://turtlebot_le2i/meshes/rplidar_main.STL" scale="0.001 0.001 0.001"/>
 			</geometry>
-			<material name="Green" />
+			<material name="blue">
+				<color rgba="0 0 .8 1"/>
+			</material>
 		</visual>
-		<inertial>
-			<mass value="0.000001" />
+		<collision>
+			<origin xyz="0.0 0.0 0.0" rpy="0 0 0"/>
+			<geometry>
+		  	      <box size="0.07271 0.27794 0.073"/>
+			</geometry>
+	  	</collision>
+	      	<inertial>
+			<mass value="0.564" />
 			<origin xyz="0 0 0" />
-			<inertia ixx="0.0001" ixy="0.0" ixz="0.0"
-			iyy="0.0001" iyz="0.0" izz="0.0001" />
-		</inertial>
+			<inertia ixx="0.003881243" ixy="0.0" ixz="0.0"
+			         iyy="0.000498940" iyz="0.0"
+			         izz="0.003879257" />
+	      	</inertial>
 	</link>
 	</xacro:macro>
